File: _saved_donut.sch (KiCad schematic (older format))
At the start: 29 parts, among them J1 AVRISP6, J2 HALL1, J3 HALL2, P1 PAD1, P2 PAD2, U1 ATMEGA48PA-MU, X1 XTAL4P

Commit message: update
Parts:
- J2, J3: footprint (none) -> Pin_Header_Straight_1x03_Pitch2.54mm
- LS1: footprint (none) -> S8211-45R
Changed lines of the file:
@@
 F 0 "LS1" H 8450 3125 50  0000 R CNN
 F 1 "Speaker" H 8450 3050 50  0000 R CNN
-F 2 "" H 8400 2700 50  0001 C CNN
+F 2 "S8211-45R" H 8400 2700 50  0001 C CNN
 F 3 "" H 8390 2850 50  0001 C CNN
 	1    8400 2900
@@
 F 0 "J2" H 1350 2500 50  0000 C CNN
 F 1 "HALL1" V 1450 2300 50  0000 C CNN
-F 2 "" H 1350 2300 50  0001 C CNN
+F 2 "Pin_Header_Straight_1x03_Pitch2.54mm" H 1350 2300 50  0001 C CNN
 F 3 "" H 1350 2300 50  0001 C CNN
 	1    1350 2300
@@
 F 0 "J3" H 1350 3000 50  0000 C CNN
 F 1 "HALL2" V 1450 2800 50  0000 C CNN
-F 2 "" H 1350 2800 50  0001 C CNN
+F 2 "Pin_Header_Straight_1x03_Pitch2.54mm" H 1350 2800 50  0001 C CNN
 F 3 "" H 1350 2800 50  0001 C CNN
 	1    1350 2800
