File: donut.sch (KiCad schematic (older format))
At the start: 29 parts, among them J1 AVRISP6, J2 HALL1, J3 HALL2, P1 PAD1, P2 PAD2, U1 ATMEGA48PA-MU, X1 XTAL4P

Commit message: Update schematic.
Parts:
- removed D1, D11, D3, D5, D7, D9: GRN, LED_0603, symbol LED
- removed D10, D12, D6, D8: RED, LED_0603, symbol LED
- removed J2: HALL1, Pin_Header_Straight_1x03_Pitch2.54mm, symbol CONN_01X03
- removed J3: HALL2, Pin_Header_Straight_1x03_Pitch2.54mm, symbol CONN_01X03
- removed RN1, RN2, RN3: 1206NETWORK, 1206NETWORK, symbol 1206NETWORK
- added BT?: Battery_Cell, S8211-45R, symbol Battery_Cell
- added C?: .33uF, C_0603, symbol C
- added J?: Jack, 3.5mm_barrel_jack_MJ-3536N, symbol Conn_01x03
- added R? (x2): 1k, R_0805, symbol R
- added R?: 100, R_0805, symbol R
- added SW? (x11): TACTILE, TACTILE10, symbol TACTILE
- added SW?: S0, TACTILE10, symbol TACTILE
- added SW?: MODE, TACTILE10, symbol TACTILE
- C2: value .1uF -> .33uF
- U1: Cost100 (none) -> 1.081; Digikey (none) -> ATMEGA168PB-AU-ND
Connections:
- net GND: now also LS1.2, BT?.2 (-), C?.2, J?.1 (Pin_1), R?.1, R?.1, SW?.3, SW?.3, SW?.3, SW?.3, SW?.3, SW?.3, SW?.3, SW?.3, SW?.3, SW?.3, SW?.3, SW?.3, SW?.3, SW?.4, SW?.4, SW?.4, SW?.4, SW?.4, SW?.4, SW?.4, SW?.4, SW?.4, SW?.4, SW?.4, SW?.4, SW?.4
- net MISO: now also SW?.1, SW?.2; no longer LS1.2
- net MOSI: now also SW?.1, SW?.2; no longer LS1.1
- net SCK: now also SW?.1, SW?.2
- net VCC: now also BT?.1 (+)
- net at U1.23 ((PCINT8/ADC0)PC0): now also P1.1
- net at D2.1 (K): now also R?.2
- net at D4.1 (K): now also R?.2
- net TSW0: now reaches U1.25 ((PCINT10/ADC2)PC2)
- net TSW0: now also SW?.1, SW?.2
- net AUD: now reaches U1.10 ((PCINT22/OC0A/AIN0)PD6)
- net AUD: now also LS1.1, U1.9 ((PCINT21/OC0B/T1)PD5), R?.2
- net TSW6: now reaches U1.2 ((PCINT20/XCK/T0)PD4)
- net TSW6: now also SW?.1, SW?.2
- net at D4.2 (A): now also D2.2 (A), U1.13 ((PCINT1/OC1A)PB1); no longer U1.26 ((PCINT11/ADC3)PC3)
- net at U1.24 ((PCINT9/ADC1)PC1): now also P2.1; no longer D2.2 (A)
- net TSW9: now reaches U1.11 ((PCINT23/AIN1)PD7)
- net TSW9: now also SW?.1, SW?.2
- net at U1.12 ((PCINT0/CLKO/ICP1)PB0): no longer P1.1
- net TSW5: now reaches U1.1 ((PCINT19/OC2B/INT1)PD3)
- net TSW5: now also SW?.1, SW?.2
- net TSW10: now reaches U1.19 (ADC6)
- net TSW10: now also SW?.1, SW?.2
- net TSW11: now reaches U1.22 (ADC7)
- net TSW11: now also SW?.1, SW?.2
- net TSW2: now reaches U1.27 ((PCINT12/SDA/ADC4)PC4)
- net TSW2: now also SW?.1, SW?.2
- net TSW3: now reaches U1.28 ((PCINT13/SCL/ADC5)PC5)
- net TSW3: now also SW?.1, SW?.2
- net RX: now reaches U1.30 ((PCINT16/RXD)PD0)
- net TX: now reaches U1.31 ((PCINT17/TXD)PD1)
- net TSW4: now reaches U1.32 ((PCINT18/INT0)PD2)
- net TSW4: now also SW?.1, SW?.2
- new net: C?.1, J?.2 (Pin_2), R?.1
- new net TSW1: SW?.1, SW?.2, U1.26 ((PCINT11/ADC3)PC3)
Other:
- note added: "(1) Mode select button.\nClick "MODE"\nClick button to switch mode."
- note added: "TODO: Figure out speaker hole diameter.\nTODO: What kind of jack for serial data?"
- moved on the sheet: D2, D4, LS1, P1, P2

Commit message: Update design
Parts:
- gave numbers to parts that had none: 19
Connections:
- net GND: no longer J2.1 (Pin_1), LS1.2, R2.1, R3.1
- net TSW5: now also U1.13 ((PCINT1/OC1A)PB1); no longer U1.1 ((PCINT19/OC2B/INT1)PD3)
- net TX: now also D2.1 (K), D4.1 (K)
- net VCC: now also R2.1, R3.1
- net at R3.2: now also D4.2 (A); no longer D4.1 (K)
- net at R2.2: now also D2.2 (A); no longer D2.1 (K)
- net TSW7: now reaches U1.12 ((PCINT0/CLKO/ICP1)PB0)
- net TSW7: now also SW8.1, SW8.2
- net MOSI renamed AUD-
- net AUD-: now also J2.1 (Pin_1), LS1.2, U1.1 ((PCINT19/OC2B/INT1)PD3); no longer SW8.1, SW8.2
Other:
- moved on the sheet: D2, D4, R2, R3

Commit message: Update donut
Parts:
- added G0: PAD1, kingdonut:kingdonut0, symbol CONN_1
- added P3, P5, P6: PAD2, SMTPIN, symbol CONN_1
- added P4: PAD1, SMTPIN, symbol CONN_1
- added SW14: TACTILE, TACTILE10Small, symbol TACTILE
- C3: value .1uF -> .33uF
- J1: footprint RIBBON6SMT -> RIBBON6SMT_POGO
- SW1, SW10, SW11, SW12, SW13, SW2, SW3, SW4, SW5, SW6, SW7, SW8, SW9: footprint TACTILE10 -> TACTILE10Small
Connections:
- net GND: now also G0.1, P3.1, P6.1, SW14.3, SW14.4
- net MISO: now also SW8.1, SW8.2; no longer SW9.1, SW9.2
- net RX: now also P4.1
- net TSW0: now also U1.28 ((PCINT13/SCL/ADC5)PC5); no longer U1.25 ((PCINT10/ADC2)PC2)
- net TSW1: now also U1.32 ((PCINT18/INT0)PD2); no longer U1.26 ((PCINT11/ADC3)PC3)
- net TSW10: now also U1.25 ((PCINT10/ADC2)PC2); no longer U1.19 (ADC6)
- net TSW11: now also U1.26 ((PCINT11/ADC3)PC3); no longer U1.22 (ADC7)
- net TSW2: now also U1.2 ((PCINT20/XCK/T0)PD4); no longer U1.27 ((PCINT12/SDA/ADC4)PC4)
- net TSW3: now also U1.6 (VCC); no longer U1.28 ((PCINT13/SCL/ADC5)PC5)
- net TSW4: now also U1.11 ((PCINT23/AIN1)PD7); no longer U1.32 ((PCINT18/INT0)PD2)
- net TSW5: now also U1.12 ((PCINT0/CLKO/ICP1)PB0); no longer U1.13 ((PCINT1/OC1A)PB1)
- net TSW6: now also U1.13 ((PCINT1/OC1A)PB1); no longer U1.2 ((PCINT20/XCK/T0)PD4)
- net TSW9: now also U1.22 (ADC7); no longer U1.11 ((PCINT23/AIN1)PD7)
- net TX: now also P5.1
- net VCC: no longer U1.6 (VCC)
- removed net TSW7: SW8.1, SW8.2, U1.12 ((PCINT0/CLKO/ICP1)PB0)
- new net TSW12: SW14.1, SW14.2, U1.27 ((PCINT12/SDA/ADC4)PC4)
- new net TSW8: SW9.1, SW9.2, U1.19 (ADC6)

Commit message: Update
Parts:
- removed LS1: Speaker, S8211-45R, symbol Speaker
- added D1, D3: NP, LED_0603, symbol LED
- added P10, P11, P12, P13, P14, P7, P9: PAD2, SMTPIN, symbol CONN_1
- added P8: PAD1, SMTPIN, symbol CONN_1
- added R4: 560, R_0805, symbol R
- added R5, R6: NP, R_0805, symbol R
- added R7, R8: 470k, R_0805, symbol R
- added U2: TSDP343xx, TO-92_Inline_Narrow_Oval, symbol TSDP343xx
- R2, R3: value 1k -> 560
- SW1: value S0 -> C
- SW10: value TACTILE -> A
- SW11: value TACTILE -> A#
- SW12: value TACTILE -> B
- SW14: value TACTILE -> C'
- SW2: value TACTILE -> C#
- SW3: value TACTILE -> D
- SW4: value TACTILE -> D#
- SW5: value TACTILE -> E
- SW6: value TACTILE -> F
- SW7: value TACTILE -> F#
- SW8: value TACTILE -> G
- SW9: value TACTILE -> G#
Connections:
- net AUD: now also P12.1
- net AUD-: now also P14.1
- net GND: now also SW1.1, SW1.2, SW10.1, SW10.2, SW11.1, SW11.2, SW12.1, SW12.2, SW13.1, SW13.2, SW2.1, SW2.2, SW3.1, SW3.2, SW4.1, SW4.2, SW5.1, SW5.2, SW6.1, SW6.2, SW7.1, SW7.2, SW8.1, SW8.2, SW9.1, SW9.2, P10.1, P9.1, U2.3 (Vs); no longer SW1.3, SW1.4, SW10.3, SW10.4, SW11.3, SW11.4, SW12.3, SW12.4, SW13.3, SW13.4, SW2.3, SW2.4, SW3.3, SW3.4, SW4.3, SW4.4, SW5.3, SW5.4, SW6.3, SW6.4, SW7.3, SW7.4, SW8.3, SW8.4, SW9.3, SW9.4
- net MISO: now also SW8.3, SW8.4; no longer SW8.1, SW8.2
- net RX: now also P8.1, U2.1 (OUT)
- net SCK: now also SW13.3, SW13.4; no longer SW13.1, SW13.2
- net TSW0: now also SW1.3, SW1.4; no longer SW1.1, SW1.2
- net TSW1: now also SW2.3, SW2.4; no longer SW2.1, SW2.2
- net TSW10: now also SW11.3, SW11.4; no longer SW11.1, SW11.2
- net TSW11: now also SW12.3, SW12.4; no longer SW12.1, SW12.2
- net TSW2: now also SW3.3, SW3.4; no longer SW3.1, SW3.2
- net TSW3: now also SW4.3, SW4.4; no longer SW4.1, SW4.2
- net TSW4: now also SW5.3, SW5.4; no longer SW5.1, SW5.2
- net TSW5: now also SW6.3, SW6.4; no longer SW6.1, SW6.2
- net TSW6: now also SW7.3, SW7.4; no longer SW7.1, SW7.2
- net TSW8: now also SW9.3, SW9.4; no longer SW9.1, SW9.2
- net TSW9: now also SW10.3, SW10.4; no longer SW10.1, SW10.2
- net TX: now also D1.1 (K), D3.1 (K), R4.2; no longer P5.1
- net VCC: now also R5.1, R6.1, R7.1, R8.1, U2.2 (GND)
- net TOUCH1: now reaches U1.23 ((PCINT8/ADC0)PC0)
- net TOUCH1: now also P2.1, R7.2; no longer P1.1
- net TOUCH2: now reaches U1.24 ((PCINT9/ADC1)PC1)
- net TOUCH2: now also P1.1, R8.2; no longer P2.1
- new net: P5.1, P7.1, R4.1
- new net: P11.1, P13.1
- new net: D1.2 (A), R5.2
- new net: D3.2 (A), R6.2
Other:
- moved on the sheet: P1, P2, P5, SW14

Commit message: Update donut
Connections:
- net GND: now also SW1.4, SW10.4, SW11.4, SW12.4, SW13.4, SW14.2, SW2.4, SW3.4, SW4.4, SW5.4, SW6.4, SW7.4, SW8.4, SW9.4; no longer SW1.1, SW10.1, SW11.1, SW12.1, SW13.1, SW14.3, SW2.1, SW3.1, SW4.1, SW5.1, SW6.1, SW7.1, SW8.1, SW9.1
- net MISO: now also SW8.1; no longer SW8.4
- net SCK: now also SW13.1; no longer SW13.4
- net TSW0: now also SW1.1; no longer SW1.4
- net TSW1: now also SW2.1; no longer SW2.4
- net TSW10: now also SW11.1; no longer SW11.4
- net TSW11: now also SW12.1; no longer SW12.4
- net TSW12: now also SW14.3; no longer SW14.2
- net TSW2: now also SW3.1; no longer SW3.4
- net TSW3: now also SW4.1; no longer SW4.4
- net TSW4: now also SW5.1; no longer SW5.4
- net TSW5: now also SW6.1; no longer SW6.4
- net TSW6: now also SW7.1; no longer SW7.4
- net TSW8: now also SW9.1; no longer SW9.4
- net TSW9: now also SW10.1; no longer SW10.4
Changed lines of the file:
@@
 Text GLabel 4100 2350 2    60   Input ~ 0
 TSW11
-Text GLabel 9300 2350 2    60   Input ~ 0
+Text GLabel 8700 2150 0    60   Input ~ 0
 TSW1
-Text GLabel 7750 2800 2    60   Input ~ 0
+Text GLabel 7150 2600 0    60   Input ~ 0
 TSW2
-Text GLabel 9300 2800 2    60   Input ~ 0
+Text GLabel 8700 2600 0    60   Input ~ 0
 TSW3
-Text GLabel 7750 3250 2    60   Input ~ 0
+Text GLabel 7150 3050 0    60   Input ~ 0
 TSW4
-Text GLabel 9300 3250 2    60   Input ~ 0
+Text GLabel 8700 3050 0    60   Input ~ 0
 TSW5
-Text GLabel 7750 3700 2    60   Input ~ 0
+Text GLabel 7150 3500 0    60   Input ~ 0
 TSW6
-Text GLabel 9300 3700 2    60   Input ~ 0
+Text GLabel 8700 3500 0    60   Input ~ 0
 TSW7
-Text GLabel 7750 4150 2    60   Input ~ 0
+Text GLabel 7150 3950 0    60   Input ~ 0
 TSW8
-Text GLabel 9300 4150 2    60   Input ~ 0
+Text GLabel 8700 3950 0    60   Input ~ 0
 TSW9
-Text GLabel 7750 4600 2    60   Input ~ 0
+Text GLabel 7150 4400 0    60   Input ~ 0
 TSW10
 Text GLabel 8700 4600 0    60   Input ~ 0
@@
 	1    0    0    -1
 $EndComp
-Text GLabel 7750 2350 2    60   Input ~ 0
+Text GLabel 7150 2150 0    60   Input ~ 0
 TSW0
 $Comp
@@
 Text GLabel 8700 4150 0    60   Input ~ 0
 TSW9
-Text GLabel 9300 4600 2    60   Input ~ 0
+Text GLabel 8700 4400 0    60   Input ~ 0
 TSW11
 $Comp
@@
 L GND #PWR022
 U 1 1 59F6F56D
-P 7150 2150
-F 0 "#PWR022" H 7150 1900 50  0001 C CNN
-F 1 "GND" H 7150 2000 50  0000 C CNN
-F 2 "" H 7150 2150 50  0001 C CNN
-F 3 "" H 7150 2150 50  0001 C CNN
-	1    7150 2150
-	0    1    1    0
+P 7750 2350
+F 0 "#PWR022" H 7750 2100 50  0001 C CNN
+F 1 "GND" H 7750 2200 50  0000 C CNN
+F 2 "" H 7750 2350 50  0001 C CNN
+F 3 "" H 7750 2350 50  0001 C CNN
+	1    7750 2350
+	0    -1   -1   0
 $EndComp
 $Comp
@@
 L GND #PWR024
 U 1 1 59F6F631
-P 7150 2600
-F 0 "#PWR024" H 7150 2350 50  0001 C CNN
-F 1 "GND" H 7150 2450 50  0000 C CNN
-F 2 "" H 7150 2600 50  0001 C CNN
-F 3 "" H 7150 2600 50  0001 C CNN
-	1    7150 2600
-	0    1    1    0
+P 7750 2800
+F 0 "#PWR024" H 7750 2550 50  0001 C CNN
+F 1 "GND" H 7750 2650 50  0000 C CNN
+F 2 "" H 7750 2800 50  0001 C CNN
+F 3 "" H 7750 2800 50  0001 C CNN
+	1    7750 2800
+	0    -1   -1   0
 $EndComp
 $Comp
@@
 L GND #PWR026
 U 1 1 59F6F712
-P 7150 3050
-F 0 "#PWR026" H 7150 2800 50  0001 C CNN
-F 1 "GND" H 7150 2900 50  0000 C CNN
-F 2 "" H 7150 3050 50  0001 C CNN
-F 3 "" H 7150 3050 50  0001 C CNN
-	1    7150 3050
-	0    1    1    0
+P 7750 3250
+F 0 "#PWR026" H 7750 3000 50  0001 C CNN
+F 1 "GND" H 7750 3100 50  0000 C CNN
+F 2 "" H 7750 3250 50  0001 C CNN
+F 3 "" H 7750 3250 50  0001 C CNN
+	1    7750 3250
+	0    -1   -1   0
 $EndComp
 $Comp
@@
 L GND #PWR028
 U 1 1 59F6F7D6
-P 7150 3500
-F 0 "#PWR028" H 7150 3250 50  0001 C CNN
-F 1 "GND" H 7150 3350 50  0000 C CNN
-F 2 "" H 7150 3500 50  0001 C CNN
-F 3 "" H 7150 3500 50  0001 C CNN
-	1    7150 3500
-	0    1    1    0
+P 7750 3700
+F 0 "#PWR028" H 7750 3450 50  0001 C CNN
+F 1 "GND" H 7750 3550 50  0000 C CNN
+F 2 "" H 7750 3700 50  0001 C CNN
+F 3 "" H 7750 3700 50  0001 C CNN
+	1    7750 3700
+	0    -1   -1   0
 $EndComp
 $Comp
@@
 L GND #PWR030
 U 1 1 59F6F8D4
-P 7150 3950
-F 0 "#PWR030" H 7150 3700 50  0001 C CNN
-F 1 "GND" H 7150 3800 50  0000 C CNN
-F 2 "" H 7150 3950 50  0001 C CNN
-F 3 "" H 7150 3950 50  0001 C CNN
-	1    7150 3950
-	0    1    1    0
+P 7750 4150
+F 0 "#PWR030" H 7750 3900 50  0001 C CNN
+F 1 "GND" H 7750 4000 50  0000 C CNN
+F 2 "" H 7750 4150 50  0001 C CNN
+F 3 "" H 7750 4150 50  0001 C CNN
+	1    7750 4150
+	0    -1   -1   0
 $EndComp
 $Comp
 L GND #PWR031
 U 1 1 59F6FA2E
-P 7150 4400
-F 0 "#PWR031" H 7150 4150 50  0001 C CNN
-F 1 "GND" H 7150 4250 50  0000 C CNN
-F 2 "" H 7150 4400 50  0001 C CNN
-F 3 "" H 7150 4400 50  0001 C CNN
-	1    7150 4400
-	0    1    1    0
+P 7750 4600
+F 0 "#PWR031" H 7750 4350 50  0001 C CNN
+F 1 "GND" H 7750 4450 50  0000 C CNN
+F 2 "" H 7750 4600 50  0001 C CNN
+F 3 "" H 7750 4600 50  0001 C CNN
+	1    7750 4600
+	0    -1   -1   0
 $EndComp
 $Comp
@@
 L GND #PWR034
 U 1 1 59F6FB54
-P 8700 4400
-F 0 "#PWR034" H 8700 4150 50  0001 C CNN
-F 1 "GND" H 8700 4250 50  0000 C CNN
-F 2 "" H 8700 4400 50  0001 C CNN
-F 3 "" H 8700 4400 50  0001 C CNN
-	1    8700 4400
-	0    1    1    0
+P 9300 4600
+F 0 "#PWR034" H 9300 4350 50  0001 C CNN
+F 1 "GND" H 9300 4450 50  0000 C CNN
+F 2 "" H 9300 4600 50  0001 C CNN
+F 3 "" H 9300 4600 50  0001 C CNN
+	1    9300 4600
+	0    -1   -1   0
 $EndComp
 $Comp
@@
 L GND #PWR036
 U 1 1 59F6FC18
-P 8700 3950
-F 0 "#PWR036" H 8700 3700 50  0001 C CNN
-F 1 "GND" H 8700 3800 50  0000 C CNN
-F 2 "" H 8700 3950 50  0001 C CNN
-F 3 "" H 8700 3950 50  0001 C CNN
-	1    8700 3950
-	0    1    1    0
+P 9300 4150
+F 0 "#PWR036" H 9300 3900 50  0001 C CNN
+F 1 "GND" H 9300 4000 50  0000 C CNN
+F 2 "" H 9300 4150 50  0001 C CNN
+F 3 "" H 9300 4150 50  0001 C CNN
+	1    9300 4150
+	0    -1   -1   0
 $EndComp
 $Comp
@@
 L GND #PWR038
 U 1 1 59F6FCDC
-P 8700 3500
-F 0 "#PWR038" H 8700 3250 50  0001 C CNN
-F 1 "GND" H 8700 3350 50  0000 C CNN
-F 2 "" H 8700 3500 50  0001 C CNN
-F 3 "" H 8700 3500 50  0001 C CNN
-	1    8700 3500
-	0    1    1    0
+P 9300 3700
+F 0 "#PWR038" H 9300 3450 50  0001 C CNN
+F 1 "GND" H 9300 3550 50  0000 C CNN
+F 2 "" H 9300 3700 50  0001 C CNN
+F 3 "" H 9300 3700 50  0001 C CNN
+	1    9300 3700
+	0    -1   -1   0
 $EndComp
 $Comp
 L GND #PWR039
 U 1 1 59F6FD3E
-P 8700 3050
-F 0 "#PWR039" H 8700 2800 50  0001 C CNN
-F 1 "GND" H 8700 2900 50  0000 C CNN
-F 2 "" H 8700 3050 50  0001 C CNN
-F 3 "" H 8700 3050 50  0001 C CNN
-	1    8700 3050
-	0    1    1    0
+P 9300 3250
+F 0 "#PWR039" H 9300 3000 50  0001 C CNN
+F 1 "GND" H 9300 3100 50  0000 C CNN
+F 2 "" H 9300 3250 50  0001 C CNN
+F 3 "" H 9300 3250 50  0001 C CNN
+	1    9300 3250
+	0    -1   -1   0
 $EndComp
 $Comp
@@
 L GND #PWR043
 U 1 1 59F6FF91
-P 8700 2150
-F 0 "#PWR043" H 8700 1900 50  0001 C CNN
-F 1 "GND" H 8700 2000 50  0000 C CNN
-F 2 "" H 8700 2150 50  0001 C CNN
-F 3 "" H 8700 2150 50  0001 C CNN
-	1    8700 2150
-	0    1    1    0
+P 9300 2350
+F 0 "#PWR043" H 9300 2100 50  0001 C CNN
+F 1 "GND" H 9300 2200 50  0000 C CNN
+F 2 "" H 9300 2350 50  0001 C CNN
+F 3 "" H 9300 2350 50  0001 C CNN
+	1    9300 2350
+	0    -1   -1   0
 $EndComp
 $Comp
 L GND #PWR044
 U 1 1 59F6FFF3
-P 8700 2600
-F 0 "#PWR044" H 8700 2350 50  0001 C CNN
-F 1 "GND" H 8700 2450 50  0000 C CNN
-F 2 "" H 8700 2600 50  0001 C CNN
-F 3 "" H 8700 2600 50  0001 C CNN
-	1    8700 2600
-	0    1    1    0
+P 9300 2800
+F 0 "#PWR044" H 9300 2550 50  0001 C CNN
+F 1 "GND" H 9300 2650 50  0000 C CNN
+F 2 "" H 9300 2800 50  0001 C CNN
+F 3 "" H 9300 2800 50  0001 C CNN
+	1    9300 2800
+	0    -1   -1   0
 $EndComp
 Text GLabel 8050 5350 0    60   Input ~ 0
@@
 L GND #PWR045
 U 1 1 59F70CE9
-P 8050 5150
-F 0 "#PWR045" H 8050 4900 50  0001 C CNN
-F 1 "GND" H 8050 5000 50  0000 C CNN
-F 2 "" H 8050 5150 50  0001 C CNN
-F 3 "" H 8050 5150 50  0001 C CNN
-	1    8050 5150
-	0    1    1    0
+P 8650 5350
+F 0 "#PWR045" H 8650 5100 50  0001 C CNN
+F 1 "GND" H 8650 5200 50  0000 C CNN
+F 2 "" H 8650 5350 50  0001 C CNN
+F 3 "" H 8650 5350 50  0001 C CNN
+	1    8650 5350
+	0    -1   -1   0
 $EndComp
 $Comp
@@
 	0    -1   -1   0
 $EndComp
-Text GLabel 8650 5350 2    60   Input ~ 0
+Text GLabel 8050 5150 0    60   Input ~ 0
 SCK
 $Comp
@@
 Text GLabel 9550 5250 0    60   Input ~ 0
 TSW12
-Text GLabel 10150 5250 1    60   Input ~ 0
+Text GLabel 9550 5450 0    60   Input ~ 0
 TSW12
 $Comp
@@
 L GND #PWR053
 U 1 1 59F81FEC
-P 9550 5450
-F 0 "#PWR053" H 9550 5200 50  0001 C CNN
-F 1 "GND" H 9550 5300 50  0000 C CNN
-F 2 "" H 9550 5450 50  0001 C CNN
-F 3 "" H 9550 5450 50  0001 C CNN
-	1    9550 5450
-	0    1    1    0
-$EndComp
-$Comp
+P 10150 5250
+F 0 "#PWR053" H 10150 5000 50  0001 C CNN
+F 1 "GND" H 10150 5100 50  0000 C CNN
+F 2 "" H 10150 5250 50  0001 C CNN
+F 3 "" H 10150 5250 50  0001 C CNN
+	1    10150 5250
+	0    -1   -1   0
+$EndComp
+$Comp

Commit message: Update plots
Parts:
- X1: value XTAL4P -> 12MHz
Connections:
- net AUD-: now also C6.2; no longer P14.1
- net GND: no longer C6.2
- net AUD-SW: now reaches J2.3 (Pin_3)
- net AUD-SW: now also P14.1
Changed lines of the file:
@@
 LIBS:stm32f042-lqfp32
 LIBS:attinyx61
-LIBS:nc7sz08
 LIBS:donut-cache
 EELAYER 25 0
@@
 P 5350 1400
 F 0 "X1" H 5350 1550 60  0000 C CNN
-F 1 "XTAL4P" H 5350 1250 60  0000 C CNN
+F 1 "12MHz" H 5350 1250 60  0000 C CNN
 F 2 "XTAL4P" H 5350 1400 60  0000 C CNN
 F 3 "" H 5350 1400 60  0000 C CNN
@@
 Text GLabel 4100 1300 2    60   Input ~ 0
 TSW6
-Text GLabel 4950 2350 2    60   Input ~ 0
+Text GLabel 5050 2350 2    60   Input ~ 0
 TSW7
 Text GLabel 2200 2550 0    60   Input ~ 0
@@
 	1    0    0    -1
 $EndComp
-$Comp
-L GND #PWR047
-U 1 1 59F746C6
-P 5550 3350
-F 0 "#PWR047" H 5550 3100 50  0001 C CNN
-F 1 "GND" H 5550 3200 50  0000 C CNN
-F 2 "" H 5550 3350 50  0001 C CNN
-F 3 "" H 5550 3350 50  0001 C CNN
-	1    5550 3350
-	1    0    0    -1
-$EndComp
 Text Notes 7300 5300 2    60   ~ 0
 (1) Mode select button.\nClick "MODE"\nClick button to switch mode.
@@
 TX
 $Comp
-L GND #PWR048
+L GND #PWR047
 U 1 1 59F76EC0
 P 5200 4150
-F 0 "#PWR048" H 5200 3900 50  0001 C CNN
+F 0 "#PWR047" H 5200 3900 50  0001 C CNN
 F 1 "GND" H 5200 4000 50  0000 C CNN
 F 2 "" H 5200 4150 50  0001 C CNN
@@
 	0    1    1    0
 $EndComp
-Text GLabel 5800 2550 0    60   Input ~ 0
-AUD-
+Text GLabel 5550 2550 0    60   Input ~ 0
+AUD-SW
 Text GLabel 5750 2800 0    60   Input ~ 0
 AUD-
@@
 TX
 $Comp
-L VCC #PWR049
+L VCC #PWR048
 U 1 1 59F7A236
 P 5950 4450
-F 0 "#PWR049" H 5950 4300 50  0001 C CNN
+F 0 "#PWR048" H 5950 4300 50  0001 C CNN
 F 1 "VCC" H 5950 4600 50  0000 C CNN
 F 2 "" H 5950 4450 50  0001 C CNN
@@
 $EndComp
 $Comp
-L VCC #PWR050
+L VCC #PWR049
 U 1 1 59F7A36A
 P 5950 4700
-F 0 "#PWR050" H 5950 4550 50  0001 C CNN
+F 0 "#PWR049" H 5950 4550 50  0001 C CNN
 F 1 "VCC" H 5950 4850 50  0000 C CNN
 F 2 "" H 5950 4700 50  0001 C CNN
@@
 $EndComp
 $Comp
-L GND #PWR051
+L GND #PWR050
 U 1 1 59F7ECDF
 P 6700 600
-F 0 "#PWR051" H 6700 350 50  0001 C CNN
+F 0 "#PWR050" H 6700 350 50  0001 C CNN
 F 1 "GND" H 6700 450 50  0000 C CNN
 F 2 "" H 6700 600 50  0001 C CNN
@@
 TSW12
 $Comp
-L GND #PWR052
+L GND #PWR051
 U 1 1 59F81F78
 P 10150 5450
-F 0 "#PWR052" H 10150 5200 50  0001 C CNN
+F 0 "#PWR051" H 10150 5200 50  0001 C CNN
 F 1 "GND" H 10150 5300 50  0000 C CNN
 F 2 "" H 10150 5450 50  0001 C CNN
@@
 $EndComp
 $Comp
-L GND #PWR053
+L GND #PWR052
 U 1 1 59F81FEC
 P 10150 5250
-F 0 "#PWR053" H 10150 5000 50  0001 C CNN
+F 0 "#PWR052" H 10150 5000 50  0001 C CNN
 F 1 "GND" H 10150 5100 50  0000 C CNN
 F 2 "" H 10150 5250 50  0001 C CNN
@@
 $EndComp
 $Comp
-L GND #PWR054
+L GND #PWR053
 U 1 1 59F8638E
 P 5200 3850
-F 0 "#PWR054" H 5200 3600 50  0001 C CNN
+F 0 "#PWR053" H 5200 3600 50  0001 C CNN
 F 1 "GND" H 5200 3700 50  0000 C CNN
 F 2 "" H 5200 3850 50  0001 C CNN
@@
 $EndComp
 $Comp
-L GND #PWR055
+L GND #PWR054
 U 1 1 5A0006A2
 P 4000 4850
-F 0 "#PWR055" H 4000 4600 50  0001 C CNN
+F 0 "#PWR054" H 4000 4600 50  0001 C CNN
 F 1 "GND" H 4000 4700 50  0000 C CNN
 F 2 "" H 4000 4850 50  0001 C CNN
@@
 $EndComp
 $Comp
-L GND #PWR056
+L GND #PWR055
 U 1 1 5A000788
 P 4000 5050
-F 0 "#PWR056" H 4000 4800 50  0001 C CNN
+F 0 "#PWR055" H 4000 4800 50  0001 C CNN
 F 1 "GND" H 4000 4900 50  0000 C CNN
 F 2 "" H 4000 5050 50  0001 C CNN
@@
 RX
 $Comp
-L GND #PWR057
+L GND #PWR056
 U 1 1 5A00655D
 P 5050 5600
-F 0 "#PWR057" H 5050 5350 50  0001 C CNN
+F 0 "#PWR056" H 5050 5350 50  0001 C CNN
 F 1 "GND" H 5050 5450 50  0000 C CNN
 F 2 "" H 5050 5600 50  0001 C CNN
@@
 $EndComp
 $Comp
-L VCC #PWR058
+L VCC #PWR057
 U 1 1 5A00665D
 P 5050 6000
-F 0 "#PWR058" H 5050 5850 50  0001 C CNN
+F 0 "#PWR057" H 5050 5850 50  0001 C CNN
 F 1 "VCC" H 5050 6150 50  0000 C CNN
 F 2 "" H 5050 6000 50  0001 C CNN
@@
 TX
 $Comp
-L VCC #PWR059
+L VCC #PWR058
 U 1 1 5A00A8EF
 P 2150 5300
-F 0 "#PWR059" H 2150 5150 50  0001 C CNN
+F 0 "#PWR058" H 2150 5150 50  0001 C CNN
 F 1 "VCC" H 2150 5450 50  0000 C CNN
 F 2 "" H 2150 5300 50  0001 C CNN
@@
 $EndComp
 $Comp
-L VCC #PWR060
+L VCC #PWR059
 U 1 1 5A00A8F5
 P 2150 5550
-F 0 "#PWR060" H 2150 5400 50  0001 C CNN
+F 0 "#PWR059" H 2150 5400 50  0001 C CNN
 F 1 "VCC" H 2150 5700 50  0000 C CNN
 F 2 "" H 2150 5550 50  0001 C CNN
@@
 $EndComp
 $Comp
-L VCC #PWR061
+L VCC #PWR060
 U 1 1 5A00B673
 P 6550 5950
-F 0 "#PWR061" H 6550 5800 50  0001 C CNN
+F 0 "#PWR060" H 6550 5800 50  0001 C CNN
 F 1 "VCC" H 6550 6100 50  0000 C CNN
 F 2 "" H 6550 5950 50  0001 C CNN
@@
 $EndComp
 $Comp
-L VCC #PWR062
+L VCC #PWR061
 U 1 1 5A00B720
 P 6550 6200
-F 0 "#PWR062" H 6550 6050 50  0001 C CNN
+F 0 "#PWR061" H 6550 6050 50  0001 C CNN
 F 1 "VCC" H 6550 6350 50  0000 C CNN
 F 2 "" H 6550 6200 50  0001 C CNN
@@
 Text GLabel 5900 5650 2    60   Input ~ 0
 TOUCH1
+Wire Wire Line
+	5050 2350 4950 2350
+Text GLabel 5550 3350 3    60   Input ~ 0
+AUD-
+Text GLabel 5750 3000 3    60   Input ~ 0
+AUD-SW
+Wire Wire Line
+	5550 2550 5800 2550
 $EndSCHEMATC
