File: donut.sch (KiCad schematic (older format))
At the start: 54 parts, among them J1 AVRISP6, J2 Jack, P1 PAD1, P10 PAD2, P11 PAD2, P12 PAD2, P13 PAD2, P14 PAD2, P2 PAD2, P3 PAD2, P4 PAD1, P5 PAD2, P6 PAD2, P7 PAD2, P8 PAD1, P9 PAD2, SW1 C, SW10 A, SW11 A#, SW12 B, SW13 MODE, SW14 C', SW2 C#, SW3 D, SW4 D#, SW5 E, SW6 F, SW7 F#, SW8 G, SW9 G#, U1 ATMEGA48PA-MU, U2 TSDP343xx, X1 12MHz

Commit message: Udpate schematci
Connections:
- net AUD-: now also J2.2 (Pin_2); no longer J2.1 (Pin_1)
- net at C6.1, R1.1: now also J2.1 (Pin_1); no longer J2.2 (Pin_2)
- net AUD-SW renamed AUD-SM
Other:
- moved on the sheet: J2
Changed lines of the file:
@@
 L Conn_01x03 J2
 U 1 1 59F70F6D
-P 5950 2900
-F 0 "J2" H 5950 3100 50  0000 C CNN
-F 1 "Jack" H 5950 2700 50  0000 C CNN
-F 2 "3.5mm_barrel_jack_MJ-3536N" H 5950 2900 50  0001 C CNN
-F 3 "" H 5950 2900 50  0001 C CNN
-	1    5950 2900
+P 6100 3000
+F 0 "J2" H 6100 3200 50  0000 C CNN
+F 1 "Jack" H 6100 2800 50  0000 C CNN
+F 2 "3.5mm_barrel_jack_MJ-3536N" H 6100 3000 50  0001 C CNN
+F 3 "" H 6100 3000 50  0001 C CNN
+	1    6100 3000
 	1    0    0    -1
 $EndComp
@@
 	0    1    1    0
 $EndComp
-Text GLabel 5550 2550 0    60   Input ~ 0
-AUD-SW
-Text GLabel 5750 2800 0    60   Input ~ 0
-AUD-
 Text GLabel 4900 2200 0    60   Input ~ 0
 MOSI
@@
 Text GLabel 4100 3100 2    60   Input ~ 0
 AUD-
-Wire Wire Line
-	4600 1400 4600 1800
-Wire Wire Line
-	4600 1800 4100 1800
-Wire Wire Line
-	5050 1400 4600 1400
-Wire Wire Line
-	4900 1550 5750 1550
-Wire Wire Line
-	5650 1550 5650 1400
-Wire Wire Line
-	5300 1700 5400 1700
-Wire Wire Line
-	4900 1350 4900 1400
-Connection ~ 4900 1400
-Wire Wire Line
-	5750 1550 5750 1350
-Connection ~ 5650 1550
-Wire Wire Line
-	5350 1750 5350 1700
-Connection ~ 5350 1700
-Wire Wire Line
-	5300 4700 5350 4700
-Wire Wire Line
-	5300 4450 5350 4450
-Wire Wire Line
-	5550 2900 5550 3050
-Connection ~ 5550 3000
-Wire Wire Line
-	5750 2900 5550 2900
-Wire Wire Line
-	5400 3000 5550 3000
-Wire Wire Line
-	4900 2200 5000 2200
 Text GLabel 5300 4450 0    60   Input ~ 0
 TX
@@
 	1    0    0    -1
 $EndComp
-Wire Wire Line
-	4900 1900 4900 1550
-Wire Wire Line
-	4100 1900 4900 1900
 $Comp
 L TACTILE SW14
@@
 	0    1    1    0
 $EndComp
-Wire Wire Line
-	3450 4850 3350 4850
-Wire Wire Line
-	3400 4850 3400 5050
-Wire Wire Line
-	3400 5050 3450 5050
-Connection ~ 3400 4850
 $Comp
 L LED D1
@@
 Text GLabel 1500 5550 0    60   Input ~ 0
 TX
-Wire Wire Line
-	1500 5550 1550 5550
-Wire Wire Line
-	1500 5300 1550 5300
 Text GLabel 1500 5300 0    60   Input ~ 0
 TX
@@
 Text GLabel 5900 5650 2    60   Input ~ 0
 TOUCH1
-Wire Wire Line
-	5050 2350 4950 2350
 Text GLabel 5550 3350 3    60   Input ~ 0
 AUD-
-Text GLabel 5750 3000 3    60   Input ~ 0
-AUD-SW
-Wire Wire Line
-	5550 2550 5800 2550
+Text GLabel 5900 3000 0    60   Input ~ 0
+AUD-
+Wire Wire Line
+	4600 1400 4600 1800
+Wire Wire Line
+	4600 1800 4100 1800
+Wire Wire Line
+	5050 1400 4600 1400
+Wire Wire Line
+	4900 1550 5750 1550
+Wire Wire Line
+	5650 1550 5650 1400
+Wire Wire Line
+	5300 1700 5400 1700
+Wire Wire Line
+	4900 1350 4900 1400
+Connection ~ 4900 1400
+Wire Wire Line
+	5750 1550 5750 1350
+Connection ~ 5650 1550
+Wire Wire Line
+	5350 1750 5350 1700
+Connection ~ 5350 1700
+Wire Wire Line
+	5300 4700 5350 4700
+Wire Wire Line
+	5300 4450 5350 4450
+Wire Wire Line
+	5550 2900 5550 3050
+Connection ~ 5550 3000
+Wire Wire Line
+	5550 2900 5900 2900
+Wire Wire Line
+	5400 3000 5550 3000
+Wire Wire Line
+	4900 2200 5000 2200
+Wire Wire Line
+	4900 1900 4900 1550
+Wire Wire Line
+	4100 1900 4900 1900
+Wire Wire Line
+	3450 4850 3350 4850
+Wire Wire Line
+	3400 4850 3400 5050
+Wire Wire Line
+	3400 5050 3450 5050
+Connection ~ 3400 4850
+Wire Wire Line
+	1500 5550 1550 5550
+Wire Wire Line
+	1500 5300 1550 5300
+Wire Wire Line
+	5050 2350 4950 2350
+Text GLabel 5800 2550 0    60   Input ~ 0
+AUD-SM
+Text GLabel 5900 3100 3    60   Input ~ 0
+AUD-SM
 $EndSCHEMATC
